File: pcb/orin-nano-controller/straps.kicad_sch (KiCad schematic)
At the start: 2 parts, among them IC1 SN74LVC07APWR, J3 Conn_01x12_Socket

Commit message: updates
Parts:
- removed IC1: SN74LVC07APWR, SamacSys:SOP65P640X120-14N, symbol SamacSys:SN74LVC07APWR
- removed J3: Conn_01x12_Socket, symbol Connector:Conn_01x12_Socket
