File: pcb/orin-nano-controller/orin-nano-controller.kicad_pcb (KiCad board)
At the start: 2 copper layers, 50 x 35 mm, 21 parts, among them IC1 SN74LVC2G07DBVR, IC2 SN74LVC2G07DBVR, J1 USB_C_Receptacle_USB2.0_14P, J2 Conn_ARM_JTAG_SWD_10, J3 Conn_01x12_Socket, U1 STM32G0B1KETx, U2 ADP1715ARMZ-3.3-R7

Commit message: ...
Parts:
- C1, C2, C3, C4, C5, C6, C_VBUS1, RA2, RA3, RA4, RA5: moved to B.Cu
- moved RCC2 8.85 mm to (86.0, 53.5), turned to 180 degrees
- moved RA5 2.89 mm to (105.5, 65.5), turned to 180 degrees
- moved RA3 2.83 mm to (105.5, 77.5), turned to 180 degrees
- moved RA4 2.83 mm to (105.5, 79.5), turned to 180 degrees
- moved RA2 2.77 mm to (105.5, 67.5), turned to 180 degrees
- moved C1 2.40 mm to (97.9, 79.0)
- moved C5 2.40 mm to (94.5, 79.0)
- moved C3 2.00 mm to (110.0, 78.5)
- moved C2 1.86 mm to (110.1, 66.5)
- moved C4 1.86 mm to (110.1, 72.5)
- turned C6 to 0 degrees
- turned C_VBUS1 to 0 degrees
Connections:
- RA2 pad 1: ORST -> OPWR
- RA4 pad 1: OPWR -> ORST
Routing:
- net +3V3: track 18.7 -> 0.00 mm, vias 0 -> 2
- net Net-(J1-CC2): track 0.00 -> 6.40 mm
- net NRST: track 2.36 -> 0.00 mm, vias 0 -> 1
- net Net-(J1-CC1): track 0.00 -> 2.25 mm
- net Net-(D1-I/O_2): track 10.7 -> 9.05 mm
- net ORST: vias 0 -> 1
- net OAPO: vias 0 -> 1
- net GND: vias 0 -> 5
- added copper zone on B.Cu, net GND

Commit message: ...
Parts:
- moved RA2 12.0 mm to (105.6, 79.5)
- moved RA4 12.0 mm to (105.6, 67.5)
- moved C4 1.28 mm to (108.9, 72.5)
Routing:
- net +3V3: track 0.00 -> 13.8 mm, vias 2 -> 3
- net OREC: vias 0 -> 1
- net OPWR: vias 0 -> 1
Changed lines of the file:
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@@
 	(footprint "Capacitor_SMD:C_0603_1608Metric_Pad1.08x0.95mm_HandSolder"
 		(layer "B.Cu")
-		(at 110.1375 72.5)
+		(at 108.8625 72.5)
 		(descr "Capacitor SMD 0603 (1608 Metric), square (rectangular) end terminal, IPC-7351 nominal with elongated pad for handsoldering. (Body size source: IPC-SM-782 page 76, https://www.pcb-3d.com/wordpress/wp-content/uploads/ipc-sm-782a_amendment_1_and_2.pdf), generated with kicad-footprint-generator")
 		(tags "capacitor handsolder")
@@
 	(footprint "Resistor_SMD:R_0603_1608Metric_Pad0.98x0.95mm_HandSolder"
 		(layer "B.Cu")
-		(at 105.5 79.5 180)
+		(at 105.5875 67.5 180)
 		(descr "Resistor SMD 0603 (1608 Metric), square (rectangular) end terminal, IPC-7351 nominal with elongated pad for handsoldering. (Body size source: IPC-SM-782 page 72, https://www.pcb-3d.com/wordpress/wp-content/uploads/ipc-sm-782a_amendment_1_and_2.pdf), generated with kicad-footprint-generator")
 		(tags "resistor handsolder")
@@
 	(footprint "Resistor_SMD:R_0603_1608Metric_Pad0.98x0.95mm_HandSolder"
 		(layer "B.Cu")
-		(at 105.5 67.5 180)
+		(at 105.5875 79.5 180)
 		(descr "Resistor SMD 0603 (1608 Metric), square (rectangular) end terminal, IPC-7351 nominal with elongated pad for handsoldering. (Body size source: IPC-SM-782 page 72, https://www.pcb-3d.com/wordpress/wp-content/uploads/ipc-sm-782a_amendment_1_and_2.pdf), generated with kicad-footprint-generator")
 		(tags "resistor handsolder")
@@
 		(net 3)
 	)
+	(via
+		(at 109.1375 78.5)
+		(size 0.6)
+		(drill 0.3)
+		(layers "F.Cu" "B.Cu")
+		(net 3)
+	)
+	(segment
+		(start 108.5 78.5)
+		(end 108 78)
+		(width 0.2)
+		(layer "B.Cu")
+		(net 3)
+	)
+	(segment
+		(start 108 72.5)
+		(end 108 67)
+		(width 0.2)
+		(layer "B.Cu")
+		(net 3)
+	)
+	(segment
+		(start 108.5 66.5)
+		(end 108 67)
+		(width 0.2)
+		(layer "B.Cu")
+		(net 3)
+	)
+	(segment
+		(start 109.275 66.5)
+		(end 108.5 66.5)
+		(width 0.2)
+		(layer "B.Cu")
+		(net 3)
+	)
+	(segment
+		(start 109.1375 78.5)
+		(end 108.5 78.5)
+		(width 0.2)
+		(layer "B.Cu")
+		(net 3)
+	)
+	(segment
+		(start 108 78)
+		(end 108 72.5)
+		(width 0.2)
+		(layer "B.Cu")
+		(net 3)
+	)
 	(segment
 		(start 94.05 67.4)
@@
 	)
 	(via
-		(at 106.4125 67.5)
+		(at 106.5 67.5)
 		(size 0.6)
 		(drill 0.3)
@@
 		(net 11)
 	)
-	(segment
+	(via
+		(at 106.5 79.5)
+		(size 0.6)
+		(drill 0.3)
+		(layers "F.Cu" "B.Cu")
+		(net 13)
+	)
+	(via
+		(at 106.4125 77.5)
+		(size 0.6)
+		(drill 0.3)
+		(layers "F.Cu" "B.Cu")
+		(net 15)
+	)
+	(segment

Commit message: ...
Parts:
- added C7: 10nF, Capacitor_SMD:C_0603_1608Metric_Pad1.08x0.95mm_HandSolder, B.Cu at (86.0, 68.4)
- added C8: 2.2μF, Capacitor_SMD:C_0603_1608Metric_Pad1.08x0.95mm_HandSolder, B.Cu at (88.5, 67.1)
- added C9: 2.2μF, Capacitor_SMD:C_0603_1608Metric_Pad1.08x0.95mm_HandSolder, B.Cu at (89.0, 62.6)
- U2: value ADP1715ARMZ-3.3-R7 -> a; moved to B.Cu
- moved U2 17.3 mm to (83.7, 64.5), turned to 180 degrees
- moved RCC1 1.50 mm to (96.5, 59.4)
Connections:
- net Net-(IC1-1Y) renamed /Controller/APO_STRAP
- net Net-(IC1-2Y) renamed /Controller/RST_STRAP
- net Net-(IC2-1Y) renamed /Controller/REC_STRAP
- net Net-(IC2-2Y) renamed /Controller/PWR_STRAP
- U1 pad 11: OPWR -> ORST
- U1 pad 9: ORST -> OPWR
- U2 pad 1: unconnected-(U2-EN-Pad1) -> +5V
- U2 pad 4: unconnected-(U2-SS-Pad4) -> Net-(U2-SS)
Routing:
- net +3V3: track 13.8 -> 39.7 mm
- net +5V: track 26.5 -> 33.2 mm, vias 0 -> 1
- net GND: track 0.00 -> 2.04 mm, vias 5 -> 3
- net Net-(U2-SS): track 0.00 -> 2.02 mm
- net Net-(J1-CC1): track 2.25 -> 2.78 mm

Commit message: ...
Routing:
- net +3V3: track 39.7 -> 65.6 mm
- net +5V: track 33.2 -> 49.4 mm
- net OAPO: track 0.00 -> 13.6 mm
- net ORST: track 0.00 -> 12.2 mm
- net NRST: track 0.00 -> 11.3 mm
- net Net-(D1-I/O_1): track 0.00 -> 11.1 mm, vias 0 -> 1
- net /Controller/RST_STRAP: track 0.00 -> 9.48 mm
- net /Controller/APO_STRAP: track 0.00 -> 8.89 mm
- net /Controller/PWR_STRAP: track 0.00 -> 8.72 mm
- net /Controller/REC_STRAP: track 0.00 -> 8.60 mm
- net OPWR: track 0.00 -> 7.25 mm
- net OREC: track 0.00 -> 6.80 mm
- net SWDIO: track 0.00 -> 6.63 mm
- net SWCLK: track 0.00 -> 5.21 mm
- net GND: track 2.04 -> 7.21 mm, vias 3 -> 4
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
Commit message: ...
Parts:
- added C10: 10 nF, Capacitor_SMD:C_0603_1608Metric_Pad1.08x0.95mm_HandSolder, F.Cu at (109.6, 53.5)
- added R1: 68 kΩ, Resistor_SMD:R_0508_1220Metric_Pad1.12x2.15mm_HandSolder, F.Cu at (104.3, 61.0)
- added R2: 100 kΩ, Resistor_SMD:R_0508_1220Metric_Pad1.12x2.15mm_HandSolder, F.Cu at (109.8, 57.0)
- added R3: 100 Ω, Resistor_SMD:R_0603_1608Metric_Pad0.98x0.95mm_HandSolder, F.Cu at (98.5, 67.0)
- C_VBUS1, RCC1, RCC2: moved to F.Cu
- J1: moved to B.Cu
- moved C_VBUS1 6.36 mm to (98.5, 60.0), turned to 180 degrees
- moved J1 5.63 mm to (91.0, 56.5), turned to 0 degrees
- moved RCC1 5.61 mm to (91.0, 60.5)
- turned RCC2 to 0 degrees
Connections:
- J3 pad 1: unconnected-(J3-Pin_1-Pad1) -> GND
- J3 pad 2: unconnected-(J3-Pin_2-Pad2) -> PC_LED+
- U1 pad 17: unconnected-(U1-PB2-Pad17) -> ADC_IN10
Routing:
- net Net-(C10-Pad1): track 0.00 -> 27.8 mm
- net GND: track 7.21 -> 28.6 mm, vias 4 -> 7
- net +5V: track 49.4 -> 34.1 mm
- net PC_LED+: track 0.00 -> 14.1 mm
- net Net-(J1-CC2): track 6.40 -> 11.6 mm
- net ADC_IN10: track 0.00 -> 2.86 mm
- net Net-(J1-CC1): track 2.78 -> 3.78 mm
- net Net-(D1-I/O_1): track 11.1 -> 10.4 mm, vias 1 -> 0

Commit message: ...
Parts:
- moved U1 1.05 mm to (94.8, 74.9)
- moved R3 1.00 mm to (97.5, 67.1)
Routing:
- net +5V: track 34.1 -> 18.5 mm, vias 1 -> 0
- net +3V3: track 65.6 -> 50.1 mm, vias 3 -> 2
- net OAPO: track 13.7 -> 0.33 mm
- net ORST: track 12.2 -> 0.00 mm
- net NRST: track 11.3 -> 0.00 mm, vias 1 -> 0
- net OPWR: track 7.25 -> 0.00 mm
- net OREC: track 6.80 -> 0.14 mm
- net SWDIO: track 6.63 -> 0.00 mm
- net SWCLK: track 5.21 -> 0.00 mm
- net GND: track 28.6 -> 23.5 mm, vias 7 -> 5
- net SWO: track 5.08 -> 0.00 mm
- net /Controller/USB_DP: track 3.63 -> 0.00 mm
- net /Controller/USB_DM: track 3.48 -> 0.00 mm
- net Net-(C10-Pad1): track 27.8 -> 26.2 mm

Commit message: updates
Parts:
- removed C_VBUS1: 1 µF, Capacitor_SMD:C_0805_2012Metric_Pad1.18x1.45mm_HandSolder
- added R4: 33 Ω, Resistor_SMD:R_0603_1608Metric_Pad0.98x0.95mm_HandSolder, F.Cu at (103.1, 70.0)
- added R5: 33 Ω, Resistor_SMD:R_0603_1608Metric_Pad0.98x0.95mm_HandSolder, F.Cu at (103.1, 72.0)
- moved R2 9.77 mm to (113.0, 56.5), turned to -90 degrees
- moved RCC1 8.15 mm to (94.1, 52.5), turned to 180 degrees
- moved IC1 7.58 mm to (110.7, 73.5)
- moved RA0 7.58 mm to (108.4, 72.5)
- moved RA1 7.58 mm to (108.5, 74.5)
- moved C4 7.57 mm to (112.8, 73.6)
- moved C6 5.67 mm to (112.8, 76.6)
- moved U2 4.01 mm to (86.0, 61.2), turned to 90 degrees
- moved IC2 3.11 mm to (110.7, 79.7)
- moved RA2 3.11 mm to (108.4, 78.6)
- moved RA3 3.11 mm to (108.5, 80.6)
- moved C8 2.99 mm to (112.8, 79.6)
- moved R3 0.90 mm to (98.4, 67.0)
- moved U1 0.83 mm to (95.6, 75.0)
- moved R1 0.61 mm to (109.5, 56.5), turned to 90 degrees
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- renumbered C10 to C1, C6 to C10, C9 to C2, C8 to C3, C2 to C4, C7 to C5, C4 to C6, C5 to C7, C3 to C8, C1 to C9, J2 to J1, J3 to J2, J1 to J3, R2 to R1, R1 to R2, RA5 to RA0, RA4 to RA1, RA3 to RA2, RA2 to RA3, RCC2 to RCC1, RCC1 to RCC2
Connections:
- J2 pad 3: unconnected-(J3-Pin_3-Pad3) -> UART2_RXD
- J2 pad 4: unconnected-(J3-Pin_4-Pad4) -> UART2_TXD
- U1 pad 15: unconnected-(U1-PB0-Pad15) -> Net-(U1-PB0)
- U1 pad 16: unconnected-(U1-PB1-Pad16) -> Net-(U1-PB1)
Routing:
- net UART2_RXD: track 0.00 -> 17.8 mm
- net UART2_TXD: track 0.00 -> 17.6 mm
- net +5V: track 18.5 -> 30.9 mm
- net NRST: track 0.00 -> 11.8 mm, vias 0 -> 1
- net OPWR: track 0.00 -> 10.8 mm
- net OAPO: track 0.33 -> 11.1 mm
- net ORST: track 0.00 -> 10.3 mm
- net OREC: track 0.14 -> 10.4 mm
- net PC_LED+: track 14.1 -> 4.01 mm
- net +3V3: track 50.1 -> 60.1 mm, vias 2 -> 3
- net Net-(J3-CC2): track 11.6 -> 2.79 mm
- net SWDIO: track 0.00 -> 6.48 mm
- net Net-(U1-PB0): track 0.00 -> 6.20 mm
- net SWCLK: track 0.00 -> 5.06 mm
- net SWO: track 0.00 -> 4.92 mm
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- added copper zone on F.Cu, net GND
Other:
- board size 50 x 35 mm -> 38 x 35 mm

Commit message: updates
Parts:
- C4: renamed from C5; footprint Capacitor_SMD:C_0603_1608Metric_Pad1.08x0.95mm_HandSolder -> Capacitor_SMD:C_0805_2012Metric_Pad1.18x1.45mm_HandSolder
- R1, R2: footprint Resistor_SMD:R_0508_1220Metric_Pad1.12x2.15mm_HandSolder -> Resistor_SMD:R_0805_2012Metric_Pad1.20x1.40mm_HandSolder
- RCC1, RCC2: moved to B.Cu
- U2: value a -> ADP1715ARMZ-3.3-R7
- moved RCC1 11.2 mm to (104.9, 55.5), turned to -90 degrees
- moved C10 7.53 mm to (85.0, 74.1), turned to -90 degrees
- moved D1 6.67 mm to (97.9, 60.8)
- moved R3 5.72 mm to (104.0, 68.1), turned to 45 degrees
- moved RCC2 4.97 mm to (90.9, 55.5), turned to 90 degrees
- moved C6 4.90 mm to (99.1, 80.7), turned to -90 degrees
- moved J1 4.69 mm to (90.4, 73.1)
- moved R5 4.00 mm to (107.0, 71.1), turned to -135 degrees
- moved U1 3.96 mm to (99.5, 75.6)
- moved J3 3.92 mm to (94.9, 56.1)
- moved C8 3.31 mm to (100.7, 80.7), turned to -90 degrees
- moved R4 2.44 mm to (105.5, 69.6), turned to -135 degrees
- moved R2 1.48 mm to (111.5, 56.8)
- moved C5 1.43 mm to (112.8, 75.0)
- moved IC1 1.42 mm to (110.7, 75.0)
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- renumbered C4 to C5, C7 to C6, C6 to C7, C9 to C8, C8 to C9
Routing:
- net +3V3: track 60.1 -> 45.1 mm
- net +5V: track 30.9 -> 18.9 mm
- net Net-(C1-Pad1): track 23.6 -> 13.9 mm
- net GND: track 24.0 -> 14.6 mm, vias 37 -> 17
- net /Controller/USB_DP: track 3.72 -> 9.71 mm
- net /Controller/USB_DM: track 3.72 -> 9.71 mm
- net Net-(D1-I/O_2): track 10.3 -> 5.38 mm
- net Net-(D1-I/O_1): track 10.3 -> 5.38 mm
- net OAPO: track 11.1 -> 6.53 mm
- net Net-(J3-CC2): track 2.79 -> 7.14 mm
- net OPWR: track 10.8 -> 6.58 mm
- net OREC: track 10.4 -> 6.12 mm
- net ORST: track 10.3 -> 6.12 mm
- net UART2_TXD: track 17.6 -> 13.7 mm
- net Net-(J3-CC1): track 3.68 -> 6.78 mm
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