File: pcb/orin-nano-controller/orin-nano-controller.kicad_pcb (KiCad board)
At the start: 2 copper layers, 38 x 35 mm, 29 parts, among them IC1 SN74LVC2G07DBVR, IC2 SN74LVC2G07DBVR, J1 Conn_ARM_JTAG_SWD_10, J2 Conn_01x12_Socket, J3 USB_C_Receptacle_USB2.0_14P, U1 STM32G0B1KETx, U2 ADP1715ARMZ-3.3-R7

Commit message: updates
Parts:
- moved R3 0.85 mm to (103.4, 68.7)
- moved R5 0.85 mm to (106.4, 71.7)
Routing:
- net +5V: track 18.9 -> 28.4 mm, vias 0 -> 1
- net Net-(C1-Pad1): track 13.9 -> 19.7 mm
- net ADC_IN10: track 3.12 -> 2.27 mm
- net UART2_TXD: track 13.7 -> 14.5 mm
- net Net-(U1-PB1): track 3.12 -> 2.27 mm
Changed lines of the file:
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@@
 	(footprint "Resistor_SMD:R_0603_1608Metric_Pad0.98x0.95mm_HandSolder"
 		(layer "F.Cu")
-		(at 107 71.145235 -135)
+		(at 106.404765 71.745235 -135)
 		(descr "Resistor SMD 0603 (1608 Metric), square (rectangular) end terminal, IPC-7351 nominal with elongated pad for handsoldering. (Body size source: IPC-SM-782 page 72, https://www.pcb-3d.com/wordpress/wp-content/uploads/ipc-sm-782a_amendment_1_and_2.pdf), generated with kicad-footprint-generator")
 		(tags "resistor handsolder")
@@
 	(footprint "Resistor_SMD:R_0603_1608Metric_Pad0.98x0.95mm_HandSolder"
 		(layer "F.Cu")
-		(at 104 68.145235 45)
+		(at 103.404765 68.745235 45)
 		(descr "Resistor SMD 0603 (1608 Metric), square (rectangular) end terminal, IPC-7351 nominal with elongated pad for handsoldering. (Body size source: IPC-SM-782 page 72, https://www.pcb-3d.com/wordpress/wp-content/uploads/ipc-sm-782a_amendment_1_and_2.pdf), generated with kicad-footprint-generator")
 		(tags "resistor handsolder")
@@
 		(net 3)
 	)
+	(via
+		(at 97.9 61.985)
+		(size 0.6)
+		(drill 0.3)
+		(layers "F.Cu" "B.Cu")
+		(net 3)
+	)
 	(segment
 		(start 88.945183 63.445183)
@@
 	)
 	(segment
+		(start 90.615 61.985)
+		(end 97.9 61.985)
+		(width 0.2)
+		(layer "B.Cu")
+		(net 3)
+	)
+	(segment
 		(start 86.975 63.445183)
 		(end 86.325 63.445183)
@@
 	)
 	(segment
+		(start 89.1 63.5)
+		(end 90.615 61.985)
+		(width 0.2)
+		(layer "B.Cu")
+		(net 3)
+	)
+	(segment
 		(start 86.975 63.445183)
 		(end 88.945183 63.445183)
@@
 	)
 	(segment
+		(start 89 63.5)
+		(end 89.1 63.5)
+		(width 0.2)
+		(layer "B.Cu")
+		(net 3)
+	)
+	(segment
 		(start 97.475 55.204346)
 		(end 97.475 54.775)
@@
 	)
 	(segment
-		(start 104.5 67.5)
+		(start 109.4 57.8)
+		(end 108.4 56.8)
+		(width 0.2)
+		(layer "F.Cu")
+		(net 37)
+	)
+	(segment
+		(start 104.05 67.95)
 		(end 109.4 62.6)
 		(width 0.2)
@@
 	)
 	(segment
-		(start 111.55 57.8)
+		(start 109.4 62.6)
 		(end 109.4 57.8)
 		(width 0.2)
@@
 	)
 	(segment
-		(start 109.4 62.6)
+		(start 111.55 57.8)
 		(end 109.4 57.8)
 		(width 0.2)
@@
 	)
 	(segment
+		(start 108.4 53.675)
+		(end 108.775 53.3)
+		(width 0.2)
+		(layer "F.Cu")
+		(net 37)
+	)
+	(segment
+		(start 108.4 56.8)
+		(end 108.4 53.675)
+		(width 0.2)
+		(layer "F.Cu")
+		(net 37)
+	)
+	(segment
+		(start 104.05 68.1)
+		(end 104.05 67.95)
+		(width 0.2)
+		(layer "F.Cu")
+		(net 37)
+	)
+	(segment
 		(start 116.96 55.8)
 		(end 117 55.84)
@@
 	)
 	(segment
-		(start 103.354765 68.79047)
-		(end 103.354765 70.41547)
+		(start 102.3 71.470235)
+		(end 102.3 69.85)
 		(width 0.2)
 		(layer "F.Cu")
@@
 	)
 	(segment
-		(start 103.354765 70.41547)
-		(end 102.3 71.470235)
+		(start 102.3 69.85)
+		(end 102.75953 69.39047)
 		(width 0.2)
 		(layer "F.Cu")
@@
 	)
 	(segment
-		(start 107.645235 70.5)
-		(end 116.6 61.545235)
+		(start 116.6 61.545235)
+		(end 116.6 61.3)
 		(width 0.2)
 		(layer "F.Cu")
@@
 	)
 	(segment
-		(start 116.6 61.3)
-		(end 117 61.3)
+		(start 107.05 71.095235)
+		(end 116.6 61.545235)
 		(width 0.2)
 		(layer "F.Cu")
@@
 	)
 	(segment
-		(start 116.6 61.545235)
-		(end 116.6 61.3)
+		(start 107.05 71.1)
+		(end 107.05 71.095235)
 		(width 0.2)
 		(layer "F.Cu")
@@
 	)
 	(segment
+		(start 116.6 61.3)
+		(end 117 61.3)
+		(width 0.2)
+		(layer "F.Cu")
+		(net 46)
+	)
+	(segment
 		(start 103.6625 53.3)
 		(end 100.155026 53.3)
@@
 	)
 	(segment
-		(start 106.354765 71.79047)
-		(end 104.729765 71.79047)
+		(start 105.304765 72.845235)
+		(end 105.75953 72.39047)
 		(width 0.2)
 		(layer "F.Cu")
@@
 	)
 	(segment
-		(start 104.729765 71.79047)
-		(end 103.675 72.845235)
+		(start 103.675 72.845235)
+		(end 105.304765 72.845235)
 		(width 0.2)
 		(layer "F.Cu")

Commit message: updates
Parts:
- added C11: 1-4.7 nF, Capacitor_SMD:C_0805_2012Metric_Pad1.18x1.45mm_HandSolder, F.Cu at (90.3, 52.0)
- added R6: 1 MΩ, Resistor_SMD:R_0805_2012Metric_Pad1.20x1.40mm_HandSolder, F.Cu at (90.3, 55.0)
- C1: footprint Capacitor_SMD:C_0603_1608Metric_Pad1.08x0.95mm_HandSolder -> Capacitor_SMD:C_0805_2012Metric_Pad1.18x1.45mm_HandSolder
- C4, U2: moved to F.Cu
- moved U2 17.8 mm to (103.8, 62.1), turned to 0 degrees
- moved C4 17.7 mm to (102.6, 65.2), turned to 0 degrees
- moved C3 13.9 mm to (102.4, 62.5), turned to 0 degrees
- moved C2 13.5 mm to (102.4, 61.0), turned to 0 degrees
- moved C10 6.85 mm to (90.4, 69.8), turned to 90 degrees
Connections:
- J3 pad A1: GND -> GNDREF
- J3 pad A12: GND -> GNDREF
- J3 pad B1: GND -> GNDREF
- J3 pad B12: GND -> GNDREF
- J3 pad S1: GND -> GNDREF
Routing:
- net +3V3: track 45.1 -> 54.3 mm
- net +5V: track 28.4 -> 21.3 mm, vias 1 -> 2
- net GND: track 14.6 -> 11.0 mm, vias 17 -> 25
- net Net-(U2-SS): track 3.17 -> 2.09 mm
- added copper zone on In1.Cu, net GND
- added copper zone on In2.Cu, net GND
- added copper zone on F.Cu, net GNDREF
Other:
- board size 38 x 35 mm -> 32.7 x 35 mm
- copper layers 2 -> 4
