File: pcb/orin-nano-controller/orin-nano-controller.kicad_pcb (KiCad board)
At the start: 4 copper layers, 32.7 x 35 mm, 31 parts, among them IC1 SN74LVC2G07DBVR, IC2 SN74LVC2G07DBVR, J1 Conn_ARM_JTAG_SWD_10, J2 Conn_01x12_Socket, J3 USB_C_Receptacle_USB2.0_14P, U1 STM32G0B1KETx, U2 ADP1715ARMZ-3.3-R7

Commit message: ../..
Parts:
- removed the C3 at (102.4, 62.5)
- added C5: 2.2μF, Capacitor_SMD:C_0805_2012Metric_Pad1.18x1.45mm_HandSolder, B.Cu at (96.3, 65.0)
- C3: renamed from C2; footprint Capacitor_SMD:C_0603_1608Metric_Pad1.08x0.95mm_HandSolder -> Capacitor_SMD:C_0805_2012Metric_Pad1.18x1.45mm_HandSolder
- C4, U2: moved to B.Cu
- RCC0: renamed from RCC1; footprint Resistor_SMD:R_0603_1608Metric_Pad0.98x0.95mm_HandSolder -> Resistor_SMD:R_0805_2012Metric_Pad1.20x1.40mm_HandSolder
- RCC1: renamed from RCC2; footprint Resistor_SMD:R_0603_1608Metric_Pad0.98x0.95mm_HandSolder -> Resistor_SMD:R_0805_2012Metric_Pad1.20x1.40mm_HandSolder
- moved U2 12.5 mm to (91.5, 64.1), turned to 180 degrees
- moved C4 10.1 mm to (92.7, 67.0), turned to 180 degrees
- moved C3 9.78 mm to (92.7, 61.1), turned to 180 degrees
- moved C1 4.17 mm to (107.3, 56.8), turned to 90 degrees
- moved C8 1.67 mm to (91.6, 70.9), turned to 0 degrees
- moved C2 0.98 mm to (90.3, 53.0)
- moved J1 0.27 mm to (90.6, 73.1)
- moved R3 0.06 mm to (90.4, 55.0)
- renumbered C8 to C10, C6 to C11, C11 to C2, C5 to C6, C10 to C8, R6 to R3, R3 to R4, R4 to R5, R5 to R6
Connections:
- J2 pad 11: unconnected-(J2-Pin_11-Pad11) -> GND
- J2 pad 7: unconnected-(J2-Pin_7-Pad7) -> GND
- J2 pad 9: unconnected-(J2-Pin_9-Pad9) -> GND
Routing:
- net +3V3: track 54.3 -> 44.5 mm
- net GND: track 11.0 -> 1.37 mm, vias 25 -> 28
- net +5V: track 21.3 -> 24.4 mm, vias 2 -> 3
- net Net-(C1-Pad1): track 19.7 -> 16.8 mm
- net GNDREF: vias 0 -> 9
- added copper zone on B.Cu, net GNDREF

Commit message: ...
Parts:
- R4, R5, R6: footprint Resistor_SMD:R_0603_1608Metric_Pad0.98x0.95mm_HandSolder -> Resistor_SMD:R_0805_2012Metric_Pad1.20x1.40mm_HandSolder
- moved R5 0.61 mm to (105.1, 70.1)
- moved R6 0.30 mm to (106.7, 71.7)
- moved R4 0.25 mm to (103.5, 68.5)
Connections:
- J3 pad A1: GNDREF -> GND
- J3 pad A12: GNDREF -> GND
- J3 pad B1: GNDREF -> GND
- J3 pad B12: GNDREF -> GND
Routing:
- net GND: track 1.37 -> 12.9 mm, vias 28 -> 41
- net +5V: track 24.4 -> 27.0 mm
- net Net-(U1-PB0): track 5.15 -> 4.48 mm

Commit message: updates
Parts:
- removed the C1 at (107.3, 56.8)
- removed the R1 at (109.4, 56.8)
- removed the R4 at (103.5, 68.5)
- added U1: TLP185xSE, Package_SO:SOIC-4_4.55x3.7mm_P2.54mm, F.Cu at (111.0, 54.5)
- C1: renamed from C2; value 1-4.7 nF -> 2.2 nF
- C6, C7: footprint Capacitor_SMD:C_0603_1608Metric_Pad1.08x0.95mm_HandSolder -> Capacitor_SMD:C_0805_2012Metric_Pad1.18x1.45mm_HandSolder
- C8: renamed from C9; footprint Capacitor_SMD:C_0603_1608Metric_Pad1.08x0.95mm_HandSolder -> Capacitor_SMD:C_0805_2012Metric_Pad1.18x1.45mm_HandSolder
- R3: renamed from R2; value 68 kΩ -> 10 kΩ
- RA0, RA1, RA2, RA3: footprint Resistor_SMD:R_0603_1608Metric_Pad0.98x0.95mm_HandSolder -> Resistor_SMD:R_0805_2012Metric_Pad1.20x1.40mm_HandSolder
- moved R3 15.9 mm to (101.3, 68.9), turned to 0 degrees
- renumbered C11 to C10, C3 to C2, C4 to C3, C5 to C4, C8 to C5, C10 to C9, R3 to R1, R5 to R2, R6 to R4, U1 to U2, U2 to U3
Connections:
- J2 pad 1: GND -> PC_LED-
- R3 pad 1: PC_LED+ -> +3V3
- R3 pad 2: Net-(C1-Pad1) -> PB2
- U2 pad 17: ADC_IN10 -> PB2
Routing:
- net PB2: track 0.00 -> 17.9 mm
- net Net-(C1-Pad1): track 16.8 -> 0.00 mm
- net +3V3: track 44.5 -> 53.5 mm, vias 3 -> 4
- net PC_LED+: track 5.47 -> 2.72 mm
- net PC_LED-: track 0.00 -> 2.71 mm
- net ADC_IN10: track 2.27 -> 0.00 mm
- net GND: vias 41 -> 40

Commit message: updates
Routing:
- net GNDREF: vias 9 -> 10
- net GND: vias 40 -> 71

Commit message: remove some vias
Routing:
- net GND: vias 71 -> 63
Changed lines of the file:
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@@
-	)
-	(via
-		(at 100.45 76.9125)
-		(size 0.6)
-		(drill 0.3)
-		(layers "F.Cu" "B.Cu")
-		(net 36)
 	)
 	(via
@@
 	)
 	(via
-		(at 102.05 74.3375)
+		(at 102.05 74.766667)
 		(size 0.6)
 		(drill 0.3)
@@
 	)
 	(via
-		(at 98.85 74.3375)
-		(size 0.6)
-		(drill 0.3)
-		(layers "F.Cu" "B.Cu")
-		(net 36)
-	)
-	(via
-		(at 100.45 74.3375)
+		(at 99.65 74.766667)
 		(size 0.6)
 		(drill 0.3)
@@
 	)
 	(via
-		(at 98.85 75.625)
-		(size 0.6)
-		(drill 0.3)
-		(layers "F.Cu" "B.Cu")
-		(net 36)
-	)
-	(via
 		(at 113.6375 75.025)
 		(size 0.6)
@@
 	)
 	(via
-		(at 100.45 78.2)
-		(size 0.6)
-		(drill 0.3)
-		(layers "F.Cu" "B.Cu")
-		(net 36)
-	)
-	(via
 		(at 118.85 58.4)
 		(size 0.6)
@@
 	)
 	(via
-		(at 97.25 75.625)
-		(size 0.6)
-		(drill 0.3)
-		(layers "F.Cu" "B.Cu")
-		(net 36)
-	)
-	(via
 		(at 104.5 51.15)
 		(size 0.6)
@@
 	)
 	(via
-		(at 100.45 75.625)
-		(size 0.6)
-		(drill 0.3)
-		(layers "F.Cu" "B.Cu")
-		(net 36)
-	)
-	(via
-		(at 98.85 78.2)
+		(at 99.65 78.2)
 		(size 0.6)
 		(drill 0.3)
@@
 	)
 	(via
-		(at 102.05 75.625)
-		(size 0.6)
-		(drill 0.3)
-		(layers "F.Cu" "B.Cu")
-		(net 36)
-	)
-	(via
 		(at 118.85 53.3)
 		(size 0.6)
@@
 	)
 	(via
-		(at 98.85 76.9125)
+		(at 99.65 76.483333)
 		(size 0.6)
 		(drill 0.3)
@@
 	)
 	(via
-		(at 102.05 76.9125)
+		(at 102.05 76.483333)
 		(size 0.6)
 		(drill 0.3)
@@
 	)
 	(via
-		(at 97.25 76.9)
-		(size 0.6)
-		(drill 0.3)
-		(layers "F.Cu" "B.Cu")
-		(net 36)
-	)
-	(via
-		(at 97.25 74.3375)
-		(size 0.6)
-		(drill 0.3)
-		(layers "F.Cu" "B.Cu")
-		(net 36)
-	)
-	(via
-		(at 100.45 73.05)
+		(at 97.2 76.5)
+		(size 0.6)
+		(drill 0.3)
+		(layers "F.Cu" "B.Cu")
+		(net 36)
+	)
+	(via
+		(at 97.2 74.75)
 		(size 0.6)
 		(drill 0.3)
@@
 	)
 	(via
-		(at 98.85 73.05)
-		(size 0.6)
-		(drill 0.3)
+		(at 99.65 73.05)
+		(size 0.6)
+		(drill 0.3)

Commit message: updates
Parts:
- C10: value 0.1 µF -> 0.1 μF

Commit message: rev 1
Parts:
- added NT1: NetTie_2, NetTie:NetTie-2_SMD_Pad0.5mm, B.Cu at (95.5, 61.0)
Connections:
- net Net-(D1-I/O_1) renamed /Frontend/USB_DM_CONN
- net Net-(D1-I/O_2) renamed /Frontend/USB_DP_CONN
- D1 pad 5: +5V -> /Frontend/VBUS_RAW
- J3 pad A4: +5V -> /Frontend/VBUS_RAW
- J3 pad A9: +5V -> /Frontend/VBUS_RAW
- J3 pad B4: +5V -> /Frontend/VBUS_RAW
- J3 pad B9: +5V -> /Frontend/VBUS_RAW
Routing:
- net /Frontend/VBUS_RAW: track 0.00 -> 23.1 mm, vias 0 -> 3
- net +5V: track 26.8 -> 3.91 mm, vias 3 -> 0
- net GND: track 12.9 -> 13.0 mm, vias 63 -> 65
Other:
- board text added: "Orin Nano Controller Rev${REVISION}"

Commit message: ...
Parts:
- C10, C9: value 0.1 μF -> 0.1 uF
- C2, C4: value 2.2μF -> 4.7 uF
- C3: value 10nF -> 10 nF
- C5: value 4.7 µF -> 4.7 uF
- C6, C8: value 0.1 µF -> 0.1 uF
- C7: value 1 µF -> 1 uF
