File: pcb/orin-nano-controller/controller.kicad_sch (KiCad schematic)
At the start: 4 parts, among them J2 Conn_ARM_JTAG_SWD_10, U1 STM32G0B1KETx

Commit message: updates
Parts:
- removed RDM, RDP: 22 Ω, Resistor_SMD:R_0603_1608Metric_Pad0.98x0.95mm_HandSolder, symbol Device:R_Small_US
- added C1: 0.1 μF, Capacitor_SMD:C_0603_1608Metric_Pad1.08x0.95mm_HandSolder, symbol Device:C_Small_US
- added C2, C3, C5: 0.1 µF, Capacitor_SMD:C_0603_1608Metric_Pad1.08x0.95mm_HandSolder, symbol Device:C_Small_US
- added C4: 1 µF, Capacitor_SMD:C_0603_1608Metric_Pad1.08x0.95mm_HandSolder, symbol Device:C_Small_US
- added C6: 4.7 µF, Capacitor_SMD:C_0805_2012Metric_Pad1.18x1.45mm_HandSolder, symbol Device:C_Small_US
- added IC1, IC2: SN74LVC2G07DBVR, SamacSys:SOT95P280X145-6N, symbol SamacSys:SN74LVC2G07DBVR
- added J3: Conn_01x12_Socket, Connector_PinSocket_2.54mm:PinSocket_1x12_P2.54mm_Horizontal, symbol Connector:Conn_01x12_Socket
- added RA2, RA3, RA4, RA5: 100 kΩ, Resistor_SMD:R_0603_1608Metric_Pad0.98x0.95mm_HandSolder, symbol Device:R_Small_US
- J2: footprint (none) -> Connector_PinHeader_1.27mm:PinHeader_2x05_P1.27mm_Vertical
Connections:
- net USB_DM: now also U1.22 (PA9/PA11)
- net USB_DP: now also U1.23 (PA10/PA12)
- net +3V3: now reaches J2.1 (VTref)
- net +3V3: now also U1.4 (VDD), C2.1, C3.1, C4.1, C5.1, C6.1, IC1.5 (VCC), IC2.5 (VCC)
- net NRST: now reaches J2.10 (~{RESET})
- net NRST: now also U1.6 (PF2), C1.1
- net SWDIO: now reaches J2.2 (SWDIO/TMS)
- net SWDIO: now also U1.24 (PA13)
- net GND: now reaches J2.3 (GND), J2.5 (GND)
- net GND: now also J2.9 (GNDDetect), U1.5 (VSS), C1.2, C2.2, C3.2, C4.2, C5.2, C6.2, IC1.2 (GND), IC2.2 (GND), RA2.2, RA3.2, RA4.2, RA5.2
- net SWCLK: now reaches J2.4 (SWCLK/TCK)
- net SWCLK: now also U1.25 (PA14)
- net SWO: now reaches J2.6 (SWO/TDO)
- net SWO: now also U1.27 (PB3)
- net OREC: now reaches U1.10 (PA3)
- net OREC: now also IC2.1 (1A), RA3.1
- net OPWR: now reaches U1.11 (PA4)
- net OPWR: now also IC2.3 (2A), RA4.1
- net OAPO: now reaches U1.12 (PA5)
- net OAPO: now also IC1.1 (1A), RA5.1
- net ORST: now reaches U1.9 (PA2)
- net ORST: now also IC1.3 (2A), RA2.1
- new net: IC1.4 (2Y), J3.8 (Pin_8)
- new net: IC1.6 (1Y), J3.5 (Pin_5)
- new net: IC2.4 (2Y), J3.12 (Pin_12)
- new net: IC2.6 (1Y), J3.10 (Pin_10)
- no-connect marks 0 -> 9
Other:
- moved on the sheet: J2, U1

Commit message: ...
Connections:
- net OPWR: now also RA2.1; no longer RA4.1
- net ORST: now also RA4.1; no longer RA2.1
- no-connect marks 9 -> 21
Other:
- moved on the sheet: RA2, RA4

Commit message: ...
Connections:
- net OPWR: now also U1.9 (PA2); no longer U1.11 (PA4)
- net ORST: now also U1.11 (PA4); no longer U1.9 (PA2)
- net RST_STRAP: now reaches IC1.4 (2Y), J3.8 (Pin_8)
- net APO_STRAP: now reaches IC1.6 (1Y), J3.5 (Pin_5)
- net PWR_STRAP: now reaches IC2.4 (2Y), J3.12 (Pin_12)
- net REC_STRAP: now reaches IC2.6 (1Y), J3.10 (Pin_10)
Other:
- moved on the sheet: RA2, RA4
Changed lines of the file:
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@@
+	)
+	(junction
+		(at 127 27.94)
+		(diameter 0)
+		(color 0 0 0 0)
+	)
+	(junction
+		(at 160.02 52.07)
+		(diameter 0)
+		(color 0 0 0 0)
 	)
 	(junction
@@
 	)
 	(junction
-		(at 165.1 52.07)
-		(diameter 0)
-		(color 0 0 0 0)
-	)
-	(junction
 		(at 215.9 67.31)
 		(diameter 0)
@@
 		(color 0 0 0 0)
 	)
-	(junction
-		(at 127 27.94)
-		(diameter 0)
-		(color 0 0 0 0)
-	)
 	(no_connect
 		(at 115.57 72.39)
@@
 	(wire
 		(pts
+			(xy 127 27.94) (xy 127 30.48)
+		)
+		(stroke
+			(width 0)
+			(type default)
+		)
+	)
+	(wire
+		(pts
+			(xy 160.02 52.07) (xy 160.02 54.61)
+		)
+		(stroke
+			(width 0)
+			(type default)
+		)
+	)
+	(wire
+		(pts
 			(xy 198.12 69.85) (xy 198.12 67.31)
 		)
@@
 	(wire
 		(pts
+			(xy 127 27.94) (xy 132.08 27.94)
+		)
+		(stroke
+			(width 0)
+			(type default)
+		)
+	)
+	(wire
+		(pts
 			(xy 184.15 119.38) (xy 190.5 119.38)
 		)
@@
 	(wire
 		(pts
-			(xy 165.1 52.07) (xy 165.1 54.61)
-		)
-		(stroke
-			(width 0)
-			(type default)
-		)
-	)
-	(wire
-		(pts
 			(xy 68.58 162.56) (xy 78.74 162.56)
 		)
@@
 	(wire
 		(pts
-			(xy 165.1 52.07) (xy 170.18 52.07)
-		)
-		(stroke
-			(width 0)
-			(type default)
-		)
-	)
-	(wire
-		(pts
 			(xy 68.58 160.02) (xy 85.09 160.02)
 		)
@@
 	(wire
 		(pts
-			(xy 149.86 52.07) (xy 165.1 52.07)
-		)
-		(stroke
-			(width 0)
-			(type default)
-		)
-	)
-	(wire
-		(pts
 			(xy 39.37 54.61) (xy 64.77 54.61)
 		)
@@
 	(wire
 		(pts
+			(xy 149.86 52.07) (xy 160.02 52.07)
+		)
+		(stroke
+			(width 0)
+			(type default)
+		)
+	)
+	(wire
+		(pts
 			(xy 200.66 148.59) (xy 200.66 151.13)
 		)
@@
 	(wire
 		(pts
-			(xy 127 27.94) (xy 127 30.48)
-		)
-		(stroke
-			(width 0)
-			(type default)
-		)
-	)
-	(wire
-		(pts
 			(xy 260.35 92.71) (xy 265.43 92.71)
 		)
@@
 	(wire
 		(pts
+			(xy 160.02 52.07) (xy 167.64 52.07)
+		)
+		(stroke
+			(width 0)
+			(type default)
+		)
+	)
+	(wire
+		(pts
 			(xy 90.17 25.4) (xy 90.17 39.37)
 		)
@@
 	(wire
 		(pts
-			(xy 127 27.94) (xy 134.62 27.94)
-		)
-		(stroke
-			(width 0)
-			(type default)
-		)
-	)
-	(wire
-		(pts
 			(xy 143.51 39.37) (xy 143.51 43.18)
 		)
@@
 			(width 0)
 			(type default)
+		)
+	)
+	(label "PWR_STRAP"
+		(at 223.52 140.97 0)
+		(effects
+			(font
+				(size 1.27 1.27)
+			)
+			(justify left bottom)
+		)
+	)
+	(label "APO_STRAP"
+		(at 242.57 74.93 0)
+		(effects
+			(font
+				(size 1.27 1.27)
+			)
+			(justify left bottom)
+		)
+	)
+	(label "REC_STRAP"
+		(at 223.52 135.89 0)
+		(effects
+			(font
+				(size 1.27 1.27)
+			)
+			(justify left bottom)
+		)
+	)
+	(label "RST_STRAP"
+		(at 237.49 88.9 0)
+		(effects
+			(font
+				(size 1.27 1.27)
+			)
+			(justify left bottom)
 		)
 	)
@@
 	(global_label "ORST"
 		(shape input)
-		(at 134.62 27.94 0)
+		(at 167.64 52.07 0)
 		(fields_autoplaced yes)
 		(effects
@@
 		)
 		(property "Intersheetrefs" "${INTERSHEET_REFS}"
-			(at 142.3828 27.94 0)
+			(at 175.4028 52.07 0)
 			(effects
 				(font
@@
 	(global_label "OPWR"
 		(shape input)
-		(at 170.18 52.07 0)
+		(at 132.08 27.94 0)
 		(fields_autoplaced yes)
 		(effects
@@
 		)
 		(property "Intersheetrefs" "${INTERSHEET_REFS}"
-			(at 178.4871 52.07 0)
+			(at 140.3871 27.94 0)
 			(effects
 				(font
@@
 	(symbol
 		(lib_id "Device:R_Small_US")
-		(at 165.1 57.15 0)
+		(at 127 33.02 0)
 		(unit 1)
 		(exclude_from_sim no)
@@
 		(fields_autoplaced yes)
 		(property "Reference" "RA2"
-			(at 167.64 55.8799 0)
+			(at 129.54 31.7499 0)
 			(effects
 				(font
@@
 		)
 		(property "Value" "100 kΩ"
-			(at 167.64 58.4199 0)
+			(at 129.54 34.2899 0)
 			(effects
 				(font
@@
 		)
 		(property "Footprint" "Resistor_SMD:R_0603_1608Metric_Pad0.98x0.95mm_HandSolder"
-			(at 165.1 57.15 0)
+			(at 127 33.02 0)
 			(effects
 				(font
@@
 		)
 		(property "Datasheet" "~"
-			(at 165.1 57.15 0)
+			(at 127 33.02 0)
 			(effects
 				(font
@@
 		)
 		(property "Description" "Resistor, small US symbol"
-			(at 165.1 57.15 0)
+			(at 127 33.02 0)
 			(effects
 				(font
@@
 	(symbol
 		(lib_id "Device:R_Small_US")
-		(at 127 33.02 0)
+		(at 160.02 57.15 0)
 		(unit 1)
 		(exclude_from_sim no)
@@
 		(fields_autoplaced yes)
 		(property "Reference" "RA4"
-			(at 129.54 31.7499 0)
+			(at 162.56 55.8799 0)
 			(effects
 				(font
@@
 		)
 		(property "Value" "100 kΩ"
-			(at 129.54 34.2899 0)
+			(at 162.56 58.4199 0)
 			(effects
 				(font
@@
 		)
 		(property "Footprint" "Resistor_SMD:R_0603_1608Metric_Pad0.98x0.95mm_HandSolder"
-			(at 127 33.02 0)
+			(at 160.02 57.15 0)
 			(effects
 				(font
@@
 		)
 		(property "Datasheet" "~"
-			(at 127 33.02 0)
+			(at 160.02 57.15 0)
 			(effects
 				(font
@@
 		)
 		(property "Description" "Resistor, small US symbol"
-			(at 127 33.02 0)
+			(at 160.02 57.15 0)
 			(effects
 				(font
@@
 	(symbol
 		(lib_id "power:GND")
-		(at 165.1 59.69 0)
+		(at 127 35.56 0)
 		(unit 1)
 		(exclude_from_sim no)
@@
 		(fields_autoplaced yes)
 		(property "Reference" "#PWR011"
-			(at 165.1 66.04 0)
+			(at 127 41.91 0)
 			(effects
 				(font
@@
 		)
 		(property "Value" "GND"
-			(at 165.1 64.77 0)
+			(at 127 40.64 0)
 			(effects
 				(font
@@
 		)
 		(property "Footprint" ""
-			(at 165.1 59.69 0)
+			(at 127 35.56 0)
 			(effects
 				(font
@@
 		)
 		(property "Datasheet" ""
-			(at 165.1 59.69 0)
+			(at 127 35.56 0)
 			(effects
 				(font
@@
 		)
 		(property "Description" "Power symbol creates a global label with name \"GND\" , ground"
-			(at 165.1 59.69 0)
+			(at 127 35.56 0)
 			(effects
 				(font
@@
 	(symbol
 		(lib_id "power:GND")
-		(at 127 35.56 0)
+		(at 160.02 59.69 0)
 		(unit 1)
 		(exclude_from_sim no)
@@
 		(fields_autoplaced yes)
 		(property "Reference" "#PWR013"
-			(at 127 41.91 0)
+			(at 160.02 66.04 0)
 			(effects
 				(font
@@
 		)
 		(property "Value" "GND"
-			(at 127 40.64 0)
+			(at 160.02 64.77 0)
 			(effects
 				(font
@@
 		)
 		(property "Footprint" ""
-			(at 127 35.56 0)
+			(at 160.02 59.69 0)
 			(effects
 				(font
@@
 		)
 		(property "Datasheet" ""
-			(at 127 35.56 0)
+			(at 160.02 59.69 0)
 			(effects
 				(font
@@
 		)
 		(property "Description" "Power symbol creates a global label with name \"GND\" , ground"
-			(at 127 35.56 0)
-			(effects
-				(font
+			(at 160.02 59.69 0)
+			(effects
+				(font

Commit message: ...
Parts:
- added C10: 10 nF, Capacitor_SMD:C_0603_1608Metric_Pad1.08x0.95mm_HandSolder, symbol Device:C_Small_US
- added R1: 68 kΩ, Resistor_SMD:R_0508_1220Metric_Pad1.12x2.15mm_HandSolder, symbol Device:R_Small_US
- added R2: 100 kΩ, Resistor_SMD:R_0508_1220Metric_Pad1.12x2.15mm_HandSolder, symbol Device:R_Small_US
- added R3: 100 Ω, Resistor_SMD:R_0603_1608Metric_Pad0.98x0.95mm_HandSolder, symbol Device:R_Small_US
Connections:
- net GND: now also J3.1 (Pin_1), C10.2, R2.2
- net PC_LED+: now reaches J3.2 (Pin_2)
- net PC_LED+: now also R1.1
- net ADC_IN10: now reaches U1.17 (PB2)
- net ADC_IN10: now also R3.1
- new net: C10.1, R1.2, R2.1, R3.2
- no-connect marks 21 -> 19

Commit message: ...
Connections:
- net UART2_RXD: now reaches J3.3 (Pin_3)
Changed lines of the file:
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@@
 	(paper "A4")
 	(junction
+		(at 242.57 74.93)
+		(diameter 0)
+		(color 0 0 0 0)
+	)
+	(junction
 		(at 90.17 39.37)
 		(diameter 0)
@@
 	(wire
 		(pts
+			(xy 242.57 77.47) (xy 242.57 74.93)
+		)
+		(stroke
+			(width 0)
+			(type default)
+		)
+	)
+	(wire
+		(pts
 			(xy 115.57 62.23) (xy 133.35 62.23)
 		)
@@
 	(wire
 		(pts
+			(xy 243.84 77.47) (xy 242.57 77.47)
+		)
+		(stroke
+			(width 0)
+			(type default)
+		)
+	)
+	(wire
+		(pts
 			(xy 143.51 -48.26) (xy 143.51 -39.37)
 		)
@@
 	(wire
 		(pts
+			(xy 242.57 74.93) (xy 265.43 74.93)
+		)
+		(stroke
+			(width 0)
+			(type default)
+		)
+	)
+	(wire
+		(pts
 			(xy 127 27.94) (xy 132.08 27.94)
 		)
@@
 	(wire
 		(pts
+			(xy 255.27 72.39) (xy 265.43 72.39)
+		)
+		(stroke
+			(width 0)
+			(type default)
+		)
+	)
+	(wire
+		(pts
 			(xy 149.86 52.07) (xy 160.02 52.07)
 		)
@@
 	(wire
 		(pts
+			(xy 255.27 69.85) (xy 265.43 69.85)
+		)
+		(stroke
+			(width 0)
+			(type default)
+		)
+	)
+	(wire
+		(pts
 			(xy 213.36 135.89) (xy 256.54 135.89)
 		)
@@
 	(wire
 		(pts
-			(xy 240.03 74.93) (xy 265.43 74.93)
+			(xy 240.03 74.93) (xy 242.57 74.93)
 		)
 		(stroke
@@
 	)
 	(label "APO_STRAP"
-		(at 242.57 74.93 0)
-		(effects
-			(font
-				(size 1.27 1.27)
-			)
-			(justify left bottom)
+		(at 243.84 77.47 0)
+		(effects
+			(font
+				(size 1.27 1.27)
+			)
+			(justify left top)
 		)
 	)
@@
 		)
 	)
+	(global_label "UART2_TXD"
+		(shape output)
+		(at 242.57 72.39 0)
+		(fields_autoplaced yes)
+		(effects
+			(font
+				(size 1.27 1.27)
+			)
+			(justify left)
+		)
+		(property "Intersheetrefs" "${INTERSHEET_REFS}"
+			(at 255.8361 72.39 0)
+			(effects
+				(font
+					(size 1.27 1.27)
+				)
+				(justify left)
+				(hide yes)
+			)
+		)
+	)
 	(global_label "OREC"
 		(shape input)
@@
 				(hide yes)
 			)
+		)
+	)
+	(global_label "UART2_RXD"
+		(shape input)
+		(at 255.27 69.85 180)
+		(fields_autoplaced yes)
+		(effects
+			(font
+				(size 1.27 1.27)
+			)
+			(justify right)
+		)
+		(property "Intersheetrefs" "${INTERSHEET_REFS}"
+			(at 241.7015 69.85 0)
+			(effects
+				(font
+					(size 1.27 1.27)
+				)
+				(justify right)
+				(hide yes)
+			)

Commit message: updates
Parts:
- added R4, R5: 33 Ω, Resistor_SMD:R_0603_1608Metric_Pad0.98x0.95mm_HandSolder, symbol Device:R_Small_US
- renumbered C10 to C1, C6 to C10, C2 to C4, C4 to C6, C5 to C7, C3 to C8, C1 to C9, J2 to J1, J3 to J2, R2 to R1, R1 to R2, RA5 to RA0, RA4 to RA1, RA3 to RA2, RA2 to RA3
Connections:
- net UART2_RXD: now also R4.1
- net UART2_TXD: now also J2.4 (Pin_4), R5.1
- net at U1.15 (PB0): now also R4.2
- net at U1.16 (PB1): now also R5.2
- no-connect marks 19 -> 17

Commit message: updates
Parts:
- R1, R2: footprint Resistor_SMD:R_0508_1220Metric_Pad1.12x2.15mm_HandSolder -> Resistor_SMD:R_0805_2012Metric_Pad1.20x1.40mm_HandSolder
- renumbered C4 to C5, C7 to C6, C6 to C7, C9 to C8, C8 to C9
Changed lines of the file:
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@@
 			)
 		)
-		(property "Footprint" "Resistor_SMD:R_0508_1220Metric_Pad1.12x2.15mm_HandSolder"
+		(property "Footprint" "Resistor_SMD:R_0805_2012Metric_Pad1.20x1.40mm_HandSolder"
 			(at 106.68 -55.88 0)
 			(effects
@@
 			)
 		)
-		(property "Datasheet" "~"
+		(property "Datasheet" ""
 			(at 106.68 -55.88 0)
 			(effects
@@
 			)
 		)
-		(property "Description" "Resistor, small US symbol"
+		(property "Description" ""
 			(at 106.68 -55.88 0)
 			(effects
@@
 			)
 		)
-		(property "Footprint" "Resistor_SMD:R_0508_1220Metric_Pad1.12x2.15mm_HandSolder"
+		(property "Footprint" "Resistor_SMD:R_0805_2012Metric_Pad1.20x1.40mm_HandSolder"
 			(at 125.73 -48.26 0)
 			(effects
@@
 			)
 		)
-		(property "Datasheet" "~"
+		(property "Datasheet" ""
 			(at 125.73 -48.26 0)
 			(effects
@@
 			)
 		)
-		(property "Description" "Resistor, small US symbol"
+		(property "Description" ""
 			(at 125.73 -48.26 0)
 			(effects
@@
 		(dnp no)
 		(fields_autoplaced yes)
-		(property "Reference" "C9"
+		(property "Reference" "C8"
 			(at 41.91 56.0069 0)
 			(effects
@@
 			(project ""
 				(path "/75c44e6f-0ea5-4980-b537-2044bb5bee98/51635310-cf84-4ff9-9fa7-4b65dd3bd30e"
-					(reference "C9")
+					(reference "C8")
 					(unit 1)
 				)
@@
 		(dnp no)
 		(fields_autoplaced yes)
-		(property "Reference" "C8"
+		(property "Reference" "C9"
 			(at 192.913 113.03 90)
 			(effects
@@
 			(project "orin-nano-controller"
 				(path "/75c44e6f-0ea5-4980-b537-2044bb5bee98/51635310-cf84-4ff9-9fa7-4b65dd3bd30e"
-					(reference "C8")
+					(reference "C9")
 					(unit 1)
 				)
@@
 		(dnp no)
 		(fields_autoplaced yes)
-		(property "Reference" "C6"
+		(property "Reference" "C7"
 			(at 208.153 44.45 90)
 			(effects
@@
 			(project ""
 				(path "/75c44e6f-0ea5-4980-b537-2044bb5bee98/51635310-cf84-4ff9-9fa7-4b65dd3bd30e"
-					(reference "C6")
+					(reference "C7")
 					(unit 1)
 				)
@@
 		(dnp no)
 		(fields_autoplaced yes)
-		(property "Reference" "C7"
+		(property "Reference" "C6"
 			(at 77.343 33.02 90)
 			(effects
@@
 			(project ""
 				(path "/75c44e6f-0ea5-4980-b537-2044bb5bee98/51635310-cf84-4ff9-9fa7-4b65dd3bd30e"
-					(reference "C7")
+					(reference "C6")
 					(unit 1)
 				)
@@
 		(dnp no)
 		(fields_autoplaced yes)
-		(property "Reference" "C4"
+		(property "Reference" "C5"
 			(at 208.153 60.96 90)
 			(effects
@@
 			(project ""
 				(path "/75c44e6f-0ea5-4980-b537-2044bb5bee98/51635310-cf84-4ff9-9fa7-4b65dd3bd30e"
-					(reference "C4")
-					(unit 1)
-				)
+					(reference "C5")
+					(unit 1)
+				)

Commit message: updates
Parts:
- C1: footprint Capacitor_SMD:C_0603_1608Metric_Pad1.08x0.95mm_HandSolder -> Capacitor_SMD:C_0805_2012Metric_Pad1.18x1.45mm_HandSolder
Changed lines of the file:
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@@
 			)
 		)
-		(property "Footprint" "Capacitor_SMD:C_0603_1608Metric_Pad1.08x0.95mm_HandSolder"
+		(property "Footprint" "Capacitor_SMD:C_0805_2012Metric_Pad1.18x1.45mm_HandSolder"
 			(at 127 -39.37 0)
 			(effects
@@
 			)
 		)
-		(property "Description" "capacitor, small US symbol"
+		(property "Description" ""
 			(at 127 -39.37 0)
 			(effects
