File: pcb/orin-nano-controller/controller.kicad_sch (KiCad schematic)
At the start: 21 parts, among them IC1 SN74LVC2G07DBVR, IC2 SN74LVC2G07DBVR, J1 Conn_ARM_JTAG_SWD_10, J2 Conn_01x12_Socket, U1 STM32G0B1KETx

Commit message: ../..
Parts:
- renumbered C8 to C10, C6 to C11, C5 to C6, C10 to C8, R3 to R4, R4 to R5, R5 to R6
Connections:
- net GND: now also J2.11 (Pin_11), J2.7 (Pin_7), J2.9 (Pin_9)
Changed lines of the file:
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@@
 		(dnp no)
 		(fields_autoplaced yes)
-		(property "Reference" "C8"
+		(property "Reference" "C10"
 			(at 41.91 56.0069 0)
 			(effects
@@
 			(project ""
 				(path "/75c44e6f-0ea5-4980-b537-2044bb5bee98/51635310-cf84-4ff9-9fa7-4b65dd3bd30e"
-					(reference "C8")
+					(reference "C10")
 					(unit 1)
 				)
@@
 		(dnp no)
 		(fields_autoplaced yes)
-		(property "Reference" "R4"
+		(property "Reference" "R5"
 			(at 45.72 63.5 90)
 			(effects
@@
 			(project ""
 				(path "/75c44e6f-0ea5-4980-b537-2044bb5bee98/51635310-cf84-4ff9-9fa7-4b65dd3bd30e"
-					(reference "R4")
+					(reference "R5")
 					(unit 1)
 				)
@@
 		(dnp no)
 		(fields_autoplaced yes)
-		(property "Reference" "R5"
+		(property "Reference" "R6"
 			(at 38.1 76.2 90)
 			(effects
@@
 			(project "orin-nano-controller"
 				(path "/75c44e6f-0ea5-4980-b537-2044bb5bee98/51635310-cf84-4ff9-9fa7-4b65dd3bd30e"
-					(reference "R5")
+					(reference "R6")
 					(unit 1)
 				)
@@
 	)
 	(symbol
+		(lib_id "power:GND")
+		(at 265.43 80.01 270)
+		(unit 1)
+		(exclude_from_sim no)
+		(in_bom yes)
+		(on_board yes)
+		(dnp no)
+		(fields_autoplaced yes)
+		(property "Reference" "#PWR031"
+			(at 259.08 80.01 0)
+			(effects
+				(font
+					(size 1.27 1.27)
+				)
+				(hide yes)
+			)
+		)
+		(property "Value" "GND"
+			(at 261.62 80.0099 90)
+			(effects
+				(font
+					(size 1.27 1.27)
+				)
+				(justify right)
+			)
+		)
+		(property "Footprint" ""
+			(at 265.43 80.01 0)
+			(effects
+				(font
+					(size 1.27 1.27)
+				)
+				(hide yes)
+			)
+		)
+		(property "Datasheet" ""
+			(at 265.43 80.01 0)
+			(effects
+				(font
+					(size 1.27 1.27)
+				)
+				(hide yes)
+			)
+		)
+		(property "Description" "Power symbol creates a global label with name \"GND\" , ground"
+			(at 265.43 80.01 0)
+			(effects
+				(font
+					(size 1.27 1.27)
+				)
+				(hide yes)
+			)
+		)
+		(pin "1"
+		)
+		(instances
+			(project ""
+				(path "/75c44e6f-0ea5-4980-b537-2044bb5bee98/51635310-cf84-4ff9-9fa7-4b65dd3bd30e"
+					(reference "#PWR031")
+					(unit 1)
+				)
+			)
+		)
+	)
+	(symbol
 		(lib_id "power:+3V3")
 		(at 215.9 35.56 0)
@@
 		(dnp no)
 		(fields_autoplaced yes)
-		(property "Reference" "R3"
+		(property "Reference" "R4"
 			(at 143.51 -60.96 90)
 			(effects
@@
 			)
 		)
-		(property "Datasheet" "~"
+		(property "Datasheet" ""
 			(at 143.51 -55.88 0)
 			(effects
@@
 			)
 		)
-		(property "Description" "Resistor, small US symbol"
+		(property "Description" ""
 			(at 143.51 -55.88 0)
 			(effects
@@
 			(project ""
 				(path "/75c44e6f-0ea5-4980-b537-2044bb5bee98/51635310-cf84-4ff9-9fa7-4b65dd3bd30e"
-					(reference "R3")
+					(reference "R4")
 					(unit 1)
 				)
@@
 	)
 	(symbol
+		(lib_id "power:GND")
+		(at 265.43 85.09 270)
+		(unit 1)
+		(exclude_from_sim no)
+		(in_bom yes)
+		(on_board yes)
+		(dnp no)
+		(fields_autoplaced yes)
+		(property "Reference" "#PWR032"
+			(at 259.08 85.09 0)
+			(effects
+				(font
+					(size 1.27 1.27)
+				)
+				(hide yes)
+			)
+		)
+		(property "Value" "GND"
+			(at 261.62 85.0899 90)
+			(effects
+				(font
+					(size 1.27 1.27)
+				)
+				(justify right)
+			)
+		)
+		(property "Footprint" ""
+			(at 265.43 85.09 0)
+			(effects
+				(font
+					(size 1.27 1.27)
+				)
+				(hide yes)
+			)
+		)
+		(property "Datasheet" ""
+			(at 265.43 85.09 0)
+			(effects
+				(font
+					(size 1.27 1.27)
+				)
+				(hide yes)
+			)
+		)
+		(property "Description" "Power symbol creates a global label with name \"GND\" , ground"
+			(at 265.43 85.09 0)
+			(effects
+				(font
+					(size 1.27 1.27)
+				)
+				(hide yes)
+			)
+		)
+		(pin "1"
+		)
+		(instances
+			(project ""
+				(path "/75c44e6f-0ea5-4980-b537-2044bb5bee98/51635310-cf84-4ff9-9fa7-4b65dd3bd30e"
+					(reference "#PWR032")
+					(unit 1)
+				)
+			)
+		)
+	)
+	(symbol
 		(lib_id "power:+3V3")
 		(at 55.88 140.97 0)
@@
 		(dnp no)
 		(fields_autoplaced yes)
-		(property "Reference" "C10"
+		(property "Reference" "C8"
 			(at 77.343 19.05 90)
 			(effects
@@
 			(project ""
 				(path "/75c44e6f-0ea5-4980-b537-2044bb5bee98/51635310-cf84-4ff9-9fa7-4b65dd3bd30e"
-					(reference "C10")
+					(reference "C8")
 					(unit 1)
 				)
@@
 		(dnp no)
 		(fields_autoplaced yes)
-		(property "Reference" "C6"
+		(property "Reference" "C11"
 			(at 77.343 33.02 90)
 			(effects
@@
 			(project ""
 				(path "/75c44e6f-0ea5-4980-b537-2044bb5bee98/51635310-cf84-4ff9-9fa7-4b65dd3bd30e"
-					(reference "C6")
+					(reference "C11")
+					(unit 1)
+				)
+			)
+		)
+	)
+	(symbol
+		(lib_id "power:GND")
+		(at 265.43 90.17 270)
+		(unit 1)
+		(exclude_from_sim no)
+		(in_bom yes)
+		(on_board yes)
+		(dnp no)
+		(fields_autoplaced yes)
+		(property "Reference" "#PWR033"
+			(at 259.08 90.17 0)
+			(effects
+				(font
+					(size 1.27 1.27)
+				)
+				(hide yes)
+			)
+		)
+		(property "Value" "GND"
+			(at 261.62 90.1699 90)
+			(effects
+				(font
+					(size 1.27 1.27)
+				)
+				(justify right)
+			)
+		)
+		(property "Footprint" ""
+			(at 265.43 90.17 0)
+			(effects
+				(font
+					(size 1.27 1.27)
+				)
+				(hide yes)
+			)
+		)
+		(property "Datasheet" ""
+			(at 265.43 90.17 0)
+			(effects
+				(font
+					(size 1.27 1.27)
+				)
+				(hide yes)
+			)
+		)
+		(property "Description" "Power symbol creates a global label with name \"GND\" , ground"
+			(at 265.43 90.17 0)
+			(effects
+				(font
+					(size 1.27 1.27)
+				)
+				(hide yes)
+			)
+		)
+		(pin "1"
+		)
+		(instances
+			(project ""
+				(path "/75c44e6f-0ea5-4980-b537-2044bb5bee98/51635310-cf84-4ff9-9fa7-4b65dd3bd30e"
+					(reference "#PWR033")
 					(unit 1)
 				)
@@
 		(dnp no)
 		(fields_autoplaced yes)
-		(property "Reference" "C5"
+		(property "Reference" "C6"
 			(at 208.153 60.96 90)
 			(effects
@@
 			(project ""
 				(path "/75c44e6f-0ea5-4980-b537-2044bb5bee98/51635310-cf84-4ff9-9fa7-4b65dd3bd30e"
-					(reference "C5")
-					(unit 1)
-				)
+					(reference "C6")
+					(unit 1)
+				)

Commit message: ...
Parts:
- R4, R5, R6: footprint Resistor_SMD:R_0603_1608Metric_Pad0.98x0.95mm_HandSolder -> Resistor_SMD:R_0805_2012Metric_Pad1.20x1.40mm_HandSolder
Changed lines of the file:
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@@
 			)
 		)
-		(property "Footprint" "Resistor_SMD:R_0603_1608Metric_Pad0.98x0.95mm_HandSolder"
+		(property "Footprint" "Resistor_SMD:R_0805_2012Metric_Pad1.20x1.40mm_HandSolder"
 			(at 45.72 69.85 0)
 			(effects
@@
 			)
 		)
-		(property "Datasheet" "~"
+		(property "Datasheet" ""
 			(at 45.72 69.85 0)
 			(effects
@@
 			)
 		)
-		(property "Description" "Resistor, small US symbol"
+		(property "Description" ""
 			(at 45.72 69.85 0)
 			(effects
@@
 			)
 		)
-		(property "Footprint" "Resistor_SMD:R_0603_1608Metric_Pad0.98x0.95mm_HandSolder"
+		(property "Footprint" "Resistor_SMD:R_0805_2012Metric_Pad1.20x1.40mm_HandSolder"
 			(at 38.1 82.55 0)
 			(effects
@@
 			)
 		)
-		(property "Datasheet" "~"
+		(property "Datasheet" ""
 			(at 38.1 82.55 0)
 			(effects
@@
 			)
 		)
-		(property "Description" "Resistor, small US symbol"
+		(property "Description" ""
 			(at 38.1 82.55 0)
 			(effects
@@
 			)
 		)
-		(property "Footprint" "Resistor_SMD:R_0603_1608Metric_Pad0.98x0.95mm_HandSolder"
+		(property "Footprint" "Resistor_SMD:R_0805_2012Metric_Pad1.20x1.40mm_HandSolder"
 			(at 143.51 -55.88 0)
 			(effects

Commit message: updates
Parts:
- removed C1: 10 nF, Capacitor_SMD:C_0805_2012Metric_Pad1.18x1.45mm_HandSolder, symbol Device:C_Small_US
- removed R1: 100 kΩ, Resistor_SMD:R_0805_2012Metric_Pad1.20x1.40mm_HandSolder, symbol Device:R_Small_US
- removed R4: 100 Ω, Resistor_SMD:R_0805_2012Metric_Pad1.20x1.40mm_HandSolder, symbol Device:R_Small_US
- added U1: TLP185xSE, Package_SO:SOIC-4_4.55x3.7mm_P2.54mm, symbol Isolator:TLP185xSE
- C6, C7: footprint Capacitor_SMD:C_0603_1608Metric_Pad1.08x0.95mm_HandSolder -> Capacitor_SMD:C_0805_2012Metric_Pad1.18x1.45mm_HandSolder
- C8: renamed from C9; footprint Capacitor_SMD:C_0603_1608Metric_Pad1.08x0.95mm_HandSolder -> Capacitor_SMD:C_0805_2012Metric_Pad1.18x1.45mm_HandSolder
- R3: renamed from R2; value 68 kΩ -> 10 kΩ
- RA0, RA1, RA2, RA3: footprint Resistor_SMD:R_0603_1608Metric_Pad0.98x0.95mm_HandSolder -> Resistor_SMD:R_0805_2012Metric_Pad1.20x1.40mm_HandSolder
- renumbered C11 to C10, C8 to C5, C10 to C9, R5 to R2, R6 to R4, U1 to U2
Connections:
- net ADC_IN10 is gone; now on net PB2: U2.17 (PB2)
- net +3V3: now also R3.1
- net GND: now also U1.4; no longer J2.1 (Pin_1)
- net PC_LED+: now also U1.1; no longer R3.1
- net PB2: now reaches R3.2
- net PB2: now also U1.6
- new net PC_LED-: J2.1 (Pin_1), U1.3
Other:
- moved on the sheet: R3

Commit message: updates
Parts:
- C10: value 0.1 µF -> 0.1 μF

Commit message: rev 1
Connections:
- no-connect marks 17 -> 19
Other:
- title: (none) -> Controller
Changed lines of the file:
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@@
 	(generator_version "9.0")
 	(paper "A4")
+	(title_block
+		(title "Controller")
+		(date "2025-10-22")
+		(rev "1")
+	)

Commit message: ...
Parts:
- C10, C9: value 0.1 μF -> 0.1 uF
- C5: value 4.7 µF -> 4.7 uF
- C6, C8: value 0.1 µF -> 0.1 uF
- C7: value 1 µF -> 1 uF
