File: pcb/orin-nano-controller/orin-nano-controller.kicad_sch (KiCad schematic)
At the start: 1 part, among them U2 AP2112K-3.3

Commit message: updates
Parts:
- removed U2: AP2112K-3.3, Package_TO_SOT_SMD:SOT-23-5, symbol Regulator_Linear:AP2112K-3.3
Other:
- removed sheet Straps
Changed lines of the file:
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@@
-		)
-	)
-	(symbol
-		(lib_id "Regulator_Linear:AP2112K-3.3")
-		(at 163.83 59.69 0)
-		(unit 1)
-		(exclude_from_sim no)
-		(in_bom yes)
-		(on_board yes)
-		(dnp no)
-		(fields_autoplaced yes)
-		(property "Reference" "U2"
-			(at 163.83 50.8 0)
-			(effects
-				(font
-					(size 1.27 1.27)
-				)
-			)
-		)
-		(property "Value" "AP2112K-3.3"
-			(at 163.83 53.34 0)
-			(effects
-				(font
-					(size 1.27 1.27)
-				)
-			)
-		)
-		(property "Footprint" "Package_TO_SOT_SMD:SOT-23-5"
-			(at 163.83 51.435 0)
-			(effects
-				(font
-					(size 1.27 1.27)
-				)
-				(hide yes)
-			)
-		)
-		(property "Datasheet" "https://www.diodes.com/assets/Datasheets/AP2112.pdf"
-			(at 163.83 57.15 0)
-			(effects
-				(font
-					(size 1.27 1.27)
-				)
-				(hide yes)
-			)
-		)
-		(property "Description" "600mA low dropout linear regulator, with enable pin, 3.8V-6V input voltage range, 3.3V fixed positive output, SOT-23-5"
-			(at 163.83 59.69 0)
-			(effects
-				(font
-					(size 1.27 1.27)
-				)
-				(hide yes)
-			)
-		)
-		(pin "1"
-		)
-		(pin "3"
-		)
-		(pin "2"
-		)
-		(pin "4"
-		)
-		(pin "5"
-		)
-		(instances
-			(project ""
-				(path "/75c44e6f-0ea5-4980-b537-2044bb5bee98"
-					(reference "U2")
-					(unit 1)
-				)
-			)
 		)
 	)
@@
 	)
 	(sheet
-		(at 160.02 123.19)
-		(size 24.13 20.32)
-		(exclude_from_sim no)
-		(in_bom yes)
-		(on_board yes)
-		(dnp no)
-		(fields_autoplaced yes)
-		(stroke
-			(width 0.1524)
-			(type solid)
-		)
-		(fill
-			(color 0 0 0 0.0000)
-		)
-		(property "Sheetname" "Straps"
-			(at 160.02 122.4784 0)
-			(effects
-				(font
-					(size 1.27 1.27)
-				)
-				(justify left bottom)
-			)
-		)
-		(property "Sheetfile" "straps.kicad_sch"
-			(at 160.02 144.0946 0)
-			(effects
-				(font
-					(size 1.27 1.27)
-				)
-				(justify left top)
-			)
-		)
-		(instances
-			(project "orin-nano-controller"
-				(path "/75c44e6f-0ea5-4980-b537-2044bb5bee98"
-					(page "4")
-				)
-			)
-		)
-	)
-	(sheet
-		(at 130.81 64.77)
+		(at 92.71 80.01)
 		(size 20.32 19.05)
 		(exclude_from_sim no)
@@
 		)
 		(property "Sheetname" "Power"
-			(at 130.81 64.0584 0)
+			(at 92.71 79.2984 0)
 			(effects
 				(font
@@
 		)
 		(property "Sheetfile" "power.kicad_sch"
-			(at 130.81 84.4046 0)
+			(at 92.71 99.6446 0)
 			(effects
 				(font
@@
 			(project "orin-nano-controller"
 				(path "/75c44e6f-0ea5-4980-b537-2044bb5bee98"
-					(page "5")
+					(page "4")
 				)
 			)

Commit message: rev 1
Other:
- title: (none) -> Jetson Orin Nano Controller
Changed lines of the file:
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@@
 	(generator_version "9.0")
 	(paper "A4")
+	(title_block
+		(title "Jetson Orin Nano Controller")
+		(date "2025-10-22")
+		(rev "1")
+	)
 	(wire
 		(pts
